File: IPRL_Sign/PCB/LED_Hub/LED_Hub/LED_Hub.kicad_pcb (KiCad board)
At the start: 2 copper layers, 97.2 x 104 mm, 49 parts, among them J1 Conn_01x02, J10 Conn_01x02, J11 Conn_01x02, J12 Conn_01x02, J13 Conn_01x02, J14 Conn_01x02, J15 Conn_01x02, J16 Conn_01x02, J17 Conn_01x02, J18 Conn_01x02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

Commit message: Added pdfs
Parts:
- added C1: 22u, Diode_SMD:D_1206_3216Metric, F.Cu at (136.8, 53.9)
- added C2: 22u, Capacitor_SMD:C_1206_3216Metric, F.Cu at (140.1, 53.8)
Routing:
- net GND: track 0.00 -> 2.02 mm, vias 0 -> 2
- added copper zone on F.Cu, net +3.3V
