File: IPRL_Sign/PCB/LED_Hub/LED_Hub/LED_Hub.kicad_sch (KiCad schematic)
At the start: 44 parts, among them J1 Conn_01x02, J10 Conn_01x02, J11 Conn_01x02, J12 Conn_01x02, J13 Conn_01x02, J14 Conn_01x02, J15 Conn_01x02, J16 Conn_01x02, J17 Conn_01x02, J18 Conn_01x02, J19 Conn_01x02, J2 Conn_01x02, J20 Conn_01x02, J21 Conn_01x02, J22 Conn_01x02, J23 Conn_01x02, J24 Conn_01x02, J25 Conn_01x02, J26 Conn_01x02, J27 Conn_01x02, J28 Conn_01x02, J29 Conn_01x02, J3 Conn_01x02, J30 Conn_01x02, J31 Conn_01x02, J32 Conn_01x02, J33 Conn_01x02, J34 Conn_01x02, J4 Conn_01x02, J5 Conn_01x02, J6 Conn_01x02, J7 Conn_01x02, J8 Conn_01x02, J9 Conn_01x02, U1 ESP32-S3-DEVKITC-1-N8R2

Commit message: Added pdfs
Parts:
- added C1: 22u, Diode_SMD:D_1206_3216Metric, symbol Device:C
- added C2: 22u, Capacitor_SMD:C_1206_3216Metric, symbol Device:C
Connections:
- net +3.3V: now also C1.1, C2.1
- net GND: now also C1.2, C2.2
Other:
- company: (none) -> Imperial Planetary Robotics lab
- title: (none) -> IPRL Sign LED Controller
