File: IPRL_2025_Ruler/PCB_RULER_IPRL_2025/PCB_RULER_IPRL_2025.kicad_pcb (KiCad board)
At the start: 2 copper layers, 155.3 x 30 mm, 48 parts, among them IC101 NT3H2211W0FTTJ, J101 USB_C_Receptacle_PowerOnly_6P, M2 MountingHole_2.2mm_M2_DIN965_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, U101 NE555D, U102 4017

Commit message: Completed IPRL Ruler 2025
Parts:
- added G***: LOGO, ruler_footprints_2025:Copper_Decal2, B.Cu at (220.5, 113.0)
- added G***: LOGO, ruler_footprints_2025:Copper_Decal, B.Cu at (214.2, 86.5)
- moved D108 6.90 mm to (104.4, 99.5)
- moved D105 6.65 mm to (97.5, 99.6)
- moved G*** 2.10 mm to (144.0, 101.0)
Routing:
- net /9: track 141.5 -> 128.6 mm
- net /4: track 134.6 -> 129.6 mm
- net /8: track 128.9 -> 130.9 mm
- net /K: track 87.7 -> 88.8 mm
Other:
- board text added: "Bolt Sizes"
- board text added: "M2"
- board text added: "Participating Countries"
